File: schema/humppakuutio.kicad_pcb (KiCad board)
At the start: 2 copper layers, 21 parts, among them P1 CONN_01X05, U1 TL074, U2 WT32

Commit message: Hardware, attempt 2
Parts:
- C1, C4, C5: footprint Capacitors_SMD:c_elec_8x6.5 -> Capacitors_ThroughHole:C_Radial_D12.5_L25_P5
- U1: moved to B.Cu
- W1, W3: footprint Wire_Pads:SolderWirePad_single_2-5mmDrill -> Wire_Pads:SolderWirePad_single_1-2mmDrill
- W2: footprint Wire_Pads:SolderWirePad_3x_2-5mmDrill -> Wire_Pads:SolderWirePad_single_1-2mmDrill
- moved W2 105.5 mm to (221.0, 94.0)
- moved W1 60.2 mm to (221.0, 88.9)
- moved C4 54.0 mm to (212.1, 90.2), turned to 180 degrees
- moved W3 42.7 mm to (221.0, 99.1)
- moved C1 35.6 mm to (191.8, 116.8)
- moved C5 35.1 mm to (210.8, 106.7), turned to 180 degrees
- moved C2 34.2 mm to (179.1, 108.0)
- moved U1 32.7 mm to (180.3, 97.8)
- moved C3 30.0 mm to (175.3, 121.9)
- moved R6 28.5 mm to (198.1, 96.5), turned to 270 degrees
- moved R3 27.2 mm to (163.8, 94.0), turned to 180 degrees
- moved P1 24.2 mm to (127.0, 92.7)
- moved U2 23.4 mm to (148.6, 99.1)
- moved R5 22.9 mm to (181.6, 116.8), turned to 90 degrees
- moved R9 21.9 mm to (175.3, 96.5), turned to 90 degrees
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Connections:
- U1 pad 1: Net-(C4-Pad2) -> Net-(C5-Pad2)
- U1 pad 2: Net-(R10-Pad2) -> Net-(R4-Pad1)
- U1 pad 3: Net-(R1-Pad1) -> Net-(R3-Pad1)
- U1 pad 5: Net-(R3-Pad1) -> Net-(R1-Pad1)
- U1 pad 6: Net-(R4-Pad1) -> Net-(R10-Pad2)
- U1 pad 7: Net-(C5-Pad2) -> Net-(C4-Pad2)
- W2 pad 1: GNDD -> GNDA
Other:
- rule pad_to_mask_clearance: 0.2 -> 0

Commit message: HW ready for making
Parts:
- moved R5 28.1 mm to (184.2, 88.9)
- moved C1 26.2 mm to (167.6, 106.7), turned to 270 degrees
- moved C2 22.6 mm to (193.0, 90.2), turned to 270 degrees
- moved C3 20.4 mm to (176.5, 101.6)
- moved R7 13.1 mm to (184.2, 82.5)
- moved R8 12.7 mm to (184.2, 94.0)
- moved R6 6.48 mm to (196.8, 90.2)
- moved C4 1.27 mm to (210.8, 90.2)
Routing:
- net VCC: track 0.00 -> 121.4 mm, vias 0 -> 2
- net GNDD: track 0.00 -> 70.1 mm, vias 0 -> 6
- net GNDA: track 0.00 -> 38.8 mm, vias 0 -> 6
- net Net-(C4-Pad2): track 0.00 -> 37.3 mm
- net Net-(C5-Pad2): track 0.00 -> 35.8 mm
- net Net-(P1-Pad3): track 0.00 -> 33.7 mm
- net Net-(P1-Pad1): track 0.00 -> 24.0 mm
- net VCOM: track 0.00 -> 23.3 mm, vias 0 -> 2
- net Net-(P1-Pad2): track 0.00 -> 22.8 mm
- net Net-(R1-Pad1): track 0.00 -> 22.5 mm
- net Net-(R10-Pad2): track 0.00 -> 21.6 mm, vias 0 -> 2
- net Net-(R3-Pad1): track 0.00 -> 18.7 mm
- net Net-(R4-Pad1): track 0.00 -> 17.5 mm
- net Net-(C5-Pad1): track 0.00 -> 13.3 mm
- net Net-(C2-Pad1): track 0.00 -> 13.2 mm
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- added copper zone on B.Cu, net GNDA
- added copper zone on B.Cu, net GNDD
Other:
- board outline added: 102.9 x 44.4 mm
- net class Default: trace_width 0.25 -> 0.4
- rule trace_min: 0.25 -> 0.4
- board text added: "HumppaKuutio 1.0"
