File: schema/humppakuutio.sch (KiCad schematic (older format))
At the start: 21 parts, among them P1 CONN_01X05, U1 TL074, U2 WT32

Commit message: Hardware, attempt 2
Parts:
- C1, C4, C5: footprint Capacitors_SMD:c_elec_8x6.5 -> Capacitors_ThroughHole:C_Radial_D12.5_L25_P5
- W1, W3: footprint Wire_Pads:SolderWirePad_single_2-5mmDrill -> Wire_Pads:SolderWirePad_single_1-2mmDrill
- W2: footprint Wire_Pads:SolderWirePad_3x_2-5mmDrill -> Wire_Pads:SolderWirePad_single_1-2mmDrill
Changed lines of the file:
@@
 $Comp
 L TL074 U1
-U 1 1 583FF90D
+U 2 1 583FF90D
 P 6900 1150
 F 0 "U1" H 6900 1350 50  0000 L CNN
@@
 F 2 "Housings_DIP:DIP-14_W7.62mm" H 6850 1250 50  0001 C CNN
 F 3 "" H 6950 1350 50  0000 C CNN
-	1    6900 1150
+	2    6900 1150
 	1    0    0    -1
 $EndComp
 $Comp
 L TL074 U1
-U 2 1 583FF9A8
+U 1 1 583FF9A8
 P 6900 2400
 F 0 "U1" H 6900 2600 50  0000 L CNN
@@
 F 2 "Housings_DIP:DIP-14_W7.62mm" H 6850 2500 50  0001 C CNN
 F 3 "" H 6950 2600 50  0000 C CNN
-	2    6900 2400
+	1    6900 2400
 	1    0    0    -1
 $EndComp
@@
 F 0 "C5" H 7675 2500 50  0000 L CNN
 F 1 "470u" H 7675 2300 50  0000 L CNN
-F 2 "Capacitors_SMD:c_elec_8x6.5" H 7688 2250 50  0001 C CNN
+F 2 "Capacitors_ThroughHole:C_Radial_D12.5_L25_P5" H 7688 2250 50  0001 C CNN
 F 3 "" H 7650 2400 50  0000 C CNN
 	1    7650 2400
@@
 F 0 "C4" H 7625 1250 50  0000 L CNN
 F 1 "470u" H 7625 1050 50  0000 L CNN
-F 2 "Capacitors_SMD:c_elec_8x6.5" H 7638 1000 50  0001 C CNN
+F 2 "Capacitors_ThroughHole:C_Radial_D12.5_L25_P5" H 7638 1000 50  0001 C CNN
 F 3 "" H 7600 1150 50  0000 C CNN
 	1    7600 1150
@@
 $EndComp
 $Comp
-L GNDD #PWR08
+L GNDA #PWR08
 U 1 1 5840342D
 P 9100 1550
 F 0 "#PWR08" H 9100 1300 50  0001 C CNN
-F 1 "GNDD" H 9100 1400 50  0000 C CNN
+F 1 "GNDA" H 9100 1400 50  0000 C CNN
 F 2 "" H 9100 1550 50  0000 C CNN
 F 3 "" H 9100 1550 50  0000 C CNN
@@
 F 0 "C1" H 4825 2550 50  0000 L CNN
 F 1 "470u" H 4825 2350 50  0000 L CNN
-F 2 "Capacitors_SMD:c_elec_8x6.5" H 4838 2300 50  0001 C CNN
+F 2 "Capacitors_ThroughHole:C_Radial_D12.5_L25_P5" H 4838 2300 50  0001 C CNN
 F 3 "" H 4800 2450 50  0000 C CNN
 	1    4800 2450
@@
 F 0 "W1" H 9400 1670 50  0001 C CNN
 F 1 "LEFT" V 9400 1600 50  0000 C CNN
-F 2 "Wire_Pads:SolderWirePad_single_2-5mmDrill" H 9600 1400 50  0001 C CNN
+F 2 "Wire_Pads:SolderWirePad_single_1-2mmDrill" H 9600 1400 50  0001 C CNN
 F 3 "" H 9600 1400 50  0000 C CNN
 	1    9400 1400
@@
 F 0 "W2" H 9400 1820 50  0001 C CNN
 F 1 "GNDA" V 9400 1750 50  0000 C CNN
-F 2 "Wire_Pads:SolderWirePad_3x_2-5mmDrill" H 9600 1550 50  0001 C CNN
+F 2 "Wire_Pads:SolderWirePad_single_1-2mmDrill" H 9600 1550 50  0001 C CNN
 F 3 "" H 9600 1550 50  0000 C CNN
 	1    9400 1550
@@
 F 0 "W3" H 9400 1970 50  0001 C CNN
 F 1 "RIGHT" V 9400 1900 50  0000 C CNN
-F 2 "Wire_Pads:SolderWirePad_single_2-5mmDrill" H 9600 1700 50  0001 C CNN
+F 2 "Wire_Pads:SolderWirePad_single_1-2mmDrill" H 9600 1700 50  0001 C CNN
 F 3 "" H 9600 1700 50  0000 C CNN
 	1    9400 1700

Commit message: Arduino Mega Shield 0.1
Parts:
- removed P1: CONN_01X05, Pin_Headers:Pin_Header_Straight_1x05, symbol CONN_01X05
- added P1: CONN_02X06, symbol CONN_02X06
- added P2: CONN_01X02, symbol CONN_01X02
- added SHIELD1: ARDUINO_MEGA_SHIELD, symbol ARDUINO_MEGA_SHIELD
Connections:
- net labels added: GND
- wire segments 85 -> 123
- no-connect marks 32 -> 99
Other:
- moved on the sheet: C1, C2, C3, C4, C5, R1, R10, R2, R3, R4, R5, R6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
